Commit message: change rtabmap project

File: catkin_ws/src/my_robot/urdf/my_robot.xacro (robot description, xacro)
@@ -121,5 +121,5 @@
      <dynamics damping="1.0" friction="1.0"/>
   </joint>
-  <link name='camera'>
+  <link name='camera_link'>
     <collision name='camera_collision'>
       <origin xyz="0 0 0" rpy=" 0 0 0"/>
@@ -146,5 +146,5 @@
   <joint type="fixed" name="camera_joint">
      <origin xyz="0.2 0 0" rpy="0 0 0"/>
-     <child link="camera"/>
+     <child link="camera_link"/>
      <parent link="chassis"/>
      <axis xyz="0 1 0" rpy="0 0 0"/>
@@ -179,3 +179,10 @@
      <axis xyz="0 1 0" rpy="0 0 0"/>
   </joint>
+  <joint name="camera_optical_joint" type="fixed">
+    <origin xyz="0 0 0" rpy="-1.5707 0 -1.5707"/>
+    <parent link="camera_link"/>
+    <child link="camera_link_optical"/>
+  </joint>
+  <link name="camera_link_optical">
+  </link>
 </robot>
